Commit message: Add files via upload

File: urdf/wheelchair.hokuyo.xacro (robot description, xacro)
@@ -15,5 +15,5 @@
   <link name="laser_joint">
    <collision>
-     <origin xyz="0 0 0" rpy="0 0 0"/>
+     <origin xyz="30 0 0" rpy="0 0 0"/>
      <geometry>
         <box size="0.1 0.1 0.1"/>
@@ -28,5 +28,5 @@
    <inertial>
      <mass value="1e-5" />
-     <origin xyz="0 0 0" rpy="0 0 0"/>
+     <origin xyz="30 0 0" rpy="0 0 0"/>
      <inertia ixx="1e-6" ixy="0" ixz="0" iyy="1e-6" iyz="0" izz="1e-6" />
    </inertial>
@@ -34,5 +34,5 @@
 <gazebo reference="laser_joint">
   <sensor type="ray" name="laser">
-    <pose>0 0 0 0 0 0</pose>
+    <pose>30 0 0 0 0 0</pose>
     <visualize>false</visualize>
     <update_rate>25</update_rate>
